Commit message: Add depth camera and rewrite launch file

File: src/description/urdf/skid_robot_v3.urdf (robot description, URDF)
Before this commit: robot simulation, 8 links, 7 joints
Links:
- removed link basefoot_link
- added link base_footprint
- added link camera_link; visual box size=0.004 0.04 0.17
Joints:
- added joint camera_joint: type fixed, parent base_link, child camera_link, origin xyz=0.15 0 0.6 rpy=0 0 0
- joint base_link_jt: parent basefoot_link -> base_footprint
