Commit message: update file bringup and urdf with camera

File: src/description/urdf/my_skid_sim.urdf (robot description, URDF)
Before this commit: robot simulation, 10 links, 9 joints
Links:
- link camera_link: geometry collision box size=0.17 0.04 0.03; visual box size=0.17 0.04 0.03
Joints:
- joint camera_joint: origin xyz=0.30 0.0 0.35 rpy=0 0 0 -> xyz=0.15 0.0 0.6 rpy=0 0 0

File: src/description/urdf/skid_robot_v3.urdf (robot description, URDF)
Before this commit: robot simulation, 9 links, 8 joints
Links:
- removed link imu
- removed link lidar
- added link imu_link, mass 0.0040208; collision mesh filename=package://simulation/meshes/visual/imu_link.STL; visual mesh filename=package://simulation/meshes/visual/imu_link.STL
- added link velodyne, mass 0.60561; collision mesh filename=package://simulation/meshes/visual/velodyne.STL; visual mesh filename=package://simulation/meshes/visual/velodyne.STL
Joints:
- removed joint imu_jt
- removed joint lidar_jt
- added joint imu_link_jt: type fixed, parent base_link, child imu_link, origin xyz=0.186696441224005 0.00158367124236836 0.2805 rpy=0 0 0, axis 0 0 0
- added joint velodyne_jt: type fixed, parent base_link, child velodyne, origin xyz=0.1976 0.0041424 0.4005 rpy=0 0 0, axis 0 0 0
